File: test/avneesh_test_files/Eagle_CAD/Flex_sensor_circuits/Eagle/Wheatstone_bridge.sch (EAGLE design)
At the start: 14 parts

Commit message: Modification 1
Parts:
- R1_IF, R1_MF: value 8 kΩ -> 12 kΩ
- R1_RF: value 8 kΩ -> 15 kΩ
- R3: value 27 kΩ -> 56 kΩ
- R4: value 12 kΩ -> 33 kΩ
Changed lines of the file:
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@@
 <part name="GND1" library="supply1" library_urn="urn:adsk.eagle:library:371" deviceset="GND" device=""/>
 <part name="V_SUPPLY" library="pinhead" library_urn="urn:adsk.eagle:library:325" deviceset="PINHD-1X1" device="" package3d_urn="urn:adsk.eagle:package:22485/2"/>
-<part name="R3" library="rcl" library_urn="urn:adsk.eagle:library:334" deviceset="R-US_" device="0207/7" package3d_urn="urn:adsk.eagle:package:23493/2" value="27 kΩ"/>
-<part name="R4" library="rcl" library_urn="urn:adsk.eagle:library:334" deviceset="R-US_" device="0207/7" package3d_urn="urn:adsk.eagle:package:23493/2" value="12 kΩ"/>
+<part name="R3" library="rcl" library_urn="urn:adsk.eagle:library:334" deviceset="R-US_" device="0207/7" package3d_urn="urn:adsk.eagle:package:23493/2" value="56 kΩ"/>
+<part name="R4" library="rcl" library_urn="urn:adsk.eagle:library:334" deviceset="R-US_" device="0207/7" package3d_urn="urn:adsk.eagle:package:23493/2" value="33 kΩ"/>
 <part name="R1_LF" library="rcl" library_urn="urn:adsk.eagle:library:334" deviceset="R-US_" device="0207/7" package3d_urn="urn:adsk.eagle:package:23493/2" value="120 kΩ"/>
-<part name="R1_RF" library="rcl" library_urn="urn:adsk.eagle:library:334" deviceset="R-US_" device="0207/7" package3d_urn="urn:adsk.eagle:package:23493/2" value="8 kΩ"/>
-<part name="R1_MF" library="rcl" library_urn="urn:adsk.eagle:library:334" deviceset="R-US_" device="0207/7" package3d_urn="urn:adsk.eagle:package:23493/2" value="8 kΩ"/>
-<part name="R1_IF" library="rcl" library_urn="urn:adsk.eagle:library:334" deviceset="R-US_" device="0207/7" package3d_urn="urn:adsk.eagle:package:23493/2" value="8 kΩ"/>
+<part name="R1_RF" library="rcl" library_urn="urn:adsk.eagle:library:334" deviceset="R-US_" device="0207/7" package3d_urn="urn:adsk.eagle:package:23493/2" value="15 kΩ"/>
+<part name="R1_MF" library="rcl" library_urn="urn:adsk.eagle:library:334" deviceset="R-US_" device="0207/7" package3d_urn="urn:adsk.eagle:package:23493/2" value="12 kΩ"/>
+<part name="R1_IF" library="rcl" library_urn="urn:adsk.eagle:library:334" deviceset="R-US_" device="0207/7" package3d_urn="urn:adsk.eagle:package:23493/2" value="12 kΩ"/>
 <part name="FS_LF" library="pinhead" library_urn="urn:adsk.eagle:library:325" deviceset="PINHD-1X2" device="" package3d_urn="urn:adsk.eagle:package:22435/2"/>
 <part name="FS_RF" library="pinhead" library_urn="urn:adsk.eagle:library:325" deviceset="PINHD-1X2" device="" package3d_urn="urn:adsk.eagle:package:22435/2"/>

Commit message: Updated flex sensor circuitry for new flex sensor
Parts:
- R1_TF: value (none) -> 47 kΩ; device pinhead:PINHD-1X2 -> rcl:R-US_0207/7
- R3: value 56 kΩ -> 68 kΩ
Other:
- moved on the sheet: C1_IN
Changed lines of the file:
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@@
 <part name="GND1" library="supply1" library_urn="urn:adsk.eagle:library:371" deviceset="GND" device=""/>
 <part name="V_SUPPLY" library="pinhead" library_urn="urn:adsk.eagle:library:325" deviceset="PINHD-1X1" device="" package3d_urn="urn:adsk.eagle:package:22485/2"/>
-<part name="R3" library="rcl" library_urn="urn:adsk.eagle:library:334" deviceset="R-US_" device="0207/7" package3d_urn="urn:adsk.eagle:package:23493/2" value="56 kΩ"/>
+<part name="R3" library="rcl" library_urn="urn:adsk.eagle:library:334" deviceset="R-US_" device="0207/7" package3d_urn="urn:adsk.eagle:package:23493/2" value="68 kΩ"/>
 <part name="R4" library="rcl" library_urn="urn:adsk.eagle:library:334" deviceset="R-US_" device="0207/7" package3d_urn="urn:adsk.eagle:package:23493/2" value="33 kΩ"/>
 <part name="R1_LF" library="rcl" library_urn="urn:adsk.eagle:library:334" deviceset="R-US_" device="0207/7" package3d_urn="urn:adsk.eagle:package:23493/2" value="120 kΩ"/>
@@
 <part name="FS_IF" library="pinhead" library_urn="urn:adsk.eagle:library:325" deviceset="PINHD-1X2" device="" package3d_urn="urn:adsk.eagle:package:22435/2"/>
 <part name="C1_IN" library="pinhead" library_urn="urn:adsk.eagle:library:325" deviceset="PINHD-1X6" device="" package3d_urn="urn:adsk.eagle:package:22472/2"/>
-<part name="R1_TF" library="pinhead" library_urn="urn:adsk.eagle:library:325" deviceset="PINHD-1X2" device="" package3d_urn="urn:adsk.eagle:package:22435/2"/>
 <part name="FS_TF" library="pinhead" library_urn="urn:adsk.eagle:library:325" deviceset="PINHD-1X2" device="" package3d_urn="urn:adsk.eagle:package:22435/2"/>
+<part name="R1_TF" library="rcl" library_urn="urn:adsk.eagle:library:334" deviceset="R-US_" device="0207/7" package3d_urn="urn:adsk.eagle:package:23493/2" value="47 kΩ"/>
 </parts>
 <sheets>
@@
 <attribute name="VALUE" x="100.33" y="27.94" size="1.778" layer="96" rot="R180"/>
 </instance>
-<instance part="C1_IN" gate="A" x="144.78" y="58.42" smashed="yes">
-<attribute name="NAME" x="138.43" y="69.215" size="1.778" layer="95"/>
-<attribute name="VALUE" x="138.43" y="48.26" size="1.778" layer="96"/>
-</instance>
-<instance part="R1_TF" gate="G$1" x="111.76" y="76.2" smashed="yes" rot="R180">
-<attribute name="NAME" x="118.11" y="70.485" size="1.778" layer="95" rot="R180"/>
-<attribute name="VALUE" x="118.11" y="81.28" size="1.778" layer="96" rot="R180"/>
+<instance part="C1_IN" gate="A" x="134.62" y="58.42" smashed="yes">
+<attribute name="NAME" x="128.27" y="69.215" size="1.778" layer="95"/>
+<attribute name="VALUE" x="128.27" y="48.26" size="1.778" layer="96"/>
 </instance>
 <instance part="FS_TF" gate="G$1" x="111.76" y="22.86" smashed="yes" rot="R180">
 <attribute name="NAME" x="118.11" y="17.145" size="1.778" layer="95" rot="R180"/>
 <attribute name="VALUE" x="118.11" y="27.94" size="1.778" layer="96" rot="R180"/>
+</instance>
+<instance part="R1_TF" gate="G$1" x="116.84" y="76.2" smashed="yes" rot="R90">
+<attribute name="NAME" x="115.3414" y="72.39" size="1.778" layer="95" rot="R90"/>
+<attribute name="VALUE" x="120.142" y="72.39" size="1.778" layer="96" rot="R90"/>
 </instance>
 </instances>
@@
 </busses>
 <nets>
-<net name="N$1" class="0">
-<segment>
-<pinref part="V_SUPPLY" gate="G$1" pin="1"/>
-<pinref part="R3" gate="G$1" pin="2"/>
-<wire x1="35.56" y1="91.44" x2="35.56" y2="83.82" width="0.1524" layer="91"/>
-<pinref part="R1_LF" gate="G$1" pin="2"/>
-<wire x1="35.56" y1="83.82" x2="35.56" y2="81.28" width="0.1524" layer="91"/>
-<wire x1="53.34" y1="81.28" x2="53.34" y2="83.82" width="0.1524" layer="91"/>
-<wire x1="53.34" y1="83.82" x2="35.56" y2="83.82" width="0.1524" layer="91"/>
-<junction x="35.56" y="83.82"/>
-<pinref part="R1_RF" gate="G$1" pin="2"/>
-<wire x1="68.58" y1="81.28" x2="68.58" y2="83.82" width="0.1524" layer="91"/>
-<wire x1="68.58" y1="83.82" x2="53.34" y2="83.82" width="0.1524" layer="91"/>
-<junction x="53.34" y="83.82"/>
-<pinref part="R1_MF" gate="G$1" pin="2"/>
-<wire x1="83.82" y1="81.28" x2="83.82" y2="83.82" width="0.1524" layer="91"/>
-<wire x1="83.82" y1="83.82" x2="68.58" y2="83.82" width="0.1524" layer="91"/>
-<junction x="68.58" y="83.82"/>
-<pinref part="R1_IF" gate="G$1" pin="2"/>
-<wire x1="99.06" y1="81.28" x2="99.06" y2="83.82" width="0.1524" layer="91"/>
-<wire x1="99.06" y1="83.82" x2="83.82" y2="83.82" width="0.1524" layer="91"/>
-<junction x="83.82" y="83.82"/>
-<pinref part="R1_TF" gate="G$1" pin="2"/>
-<wire x1="114.3" y1="76.2" x2="121.92" y2="76.2" width="0.1524" layer="91"/>
-<wire x1="121.92" y1="76.2" x2="121.92" y2="83.82" width="0.1524" layer="91"/>
-<wire x1="121.92" y1="83.82" x2="99.06" y2="83.82" width="0.1524" layer="91"/>
-<junction x="99.06" y="83.82"/>
-</segment>
-</net>
 <net name="N$2" class="0">
 <segment>
@@
 <pinref part="C1_IN" gate="A" pin="1"/>
 <wire x1="35.56" y1="66.04" x2="35.56" y2="25.4" width="0.1524" layer="91"/>
-<wire x1="142.24" y1="66.04" x2="35.56" y2="66.04" width="0.1524" layer="91"/>
+<wire x1="132.08" y1="66.04" x2="35.56" y2="66.04" width="0.1524" layer="91"/>
 <junction x="35.56" y="66.04"/>
 </segment>
@@
 <wire x1="99.06" y1="20.32" x2="99.06" y2="10.16" width="0.1524" layer="91"/>
 <pinref part="FS_TF" gate="G$1" pin="1"/>
-<wire x1="114.3" y1="20.32" x2="121.92" y2="20.32" width="0.1524" layer="91"/>
-<wire x1="121.92" y1="20.32" x2="121.92" y2="10.16" width="0.1524" layer="91"/>
-<wire x1="121.92" y1="10.16" x2="99.06" y2="10.16" width="0.1524" layer="91"/>
+<wire x1="114.3" y1="20.32" x2="116.84" y2="20.32" width="0.1524" layer="91"/>
+<wire x1="116.84" y1="20.32" x2="116.84" y2="10.16" width="0.1524" layer="91"/>
+<wire x1="116.84" y1="10.16" x2="99.06" y2="10.16" width="0.1524" layer="91"/>
 <junction x="99.06" y="10.16"/>
 </segment>
@@
 <wire x1="50.8" y1="22.86" x2="53.34" y2="22.86" width="0.1524" layer="91"/>
 <pinref part="C1_IN" gate="A" pin="2"/>
-<wire x1="142.24" y1="63.5" x2="53.34" y2="63.5" width="0.1524" layer="91"/>
+<wire x1="132.08" y1="63.5" x2="53.34" y2="63.5" width="0.1524" layer="91"/>
 <junction x="53.34" y="63.5"/>
 </segment>
@@
 <wire x1="66.04" y1="22.86" x2="68.58" y2="22.86" width="0.1524" layer="91"/>
 <pinref part="C1_IN" gate="A" pin="3"/>
-<wire x1="142.24" y1="60.96" x2="68.58" y2="60.96" width="0.1524" layer="91"/>
+<wire x1="132.08" y1="60.96" x2="68.58" y2="60.96" width="0.1524" layer="91"/>
 <junction x="68.58" y="60.96"/>
 </segment>
@@
 <wire x1="81.28" y1="22.86" x2="83.82" y2="22.86" width="0.1524" layer="91"/>
 <pinref part="C1_IN" gate="A" pin="4"/>
-<wire x1="142.24" y1="58.42" x2="83.82" y2="58.42" width="0.1524" layer="91"/>
+<wire x1="132.08" y1="58.42" x2="83.82" y2="58.42" width="0.1524" layer="91"/>
 <junction x="83.82" y="58.42"/>
 </segment>
@@
 <wire x1="96.52" y1="22.86" x2="99.06" y2="22.86" width="0.1524" layer="91"/>
 <pinref part="C1_IN" gate="A" pin="5"/>
-<wire x1="142.24" y1="55.88" x2="99.06" y2="55.88" width="0.1524" layer="91"/>
+<wire x1="132.08" y1="55.88" x2="99.06" y2="55.88" width="0.1524" layer="91"/>
 <junction x="99.06" y="55.88"/>
 </segment>
@@
 <net name="N$6" class="0">
 <segment>
+<pinref part="FS_TF" gate="G$1" pin="2"/>
+<wire x1="116.84" y1="53.34" x2="116.84" y2="22.86" width="0.1524" layer="91"/>
+<wire x1="116.84" y1="22.86" x2="114.3" y2="22.86" width="0.1524" layer="91"/>
+<pinref part="C1_IN" gate="A" pin="6"/>
+<wire x1="132.08" y1="53.34" x2="116.84" y2="53.34" width="0.1524" layer="91"/>
 <pinref part="R1_TF" gate="G$1" pin="1"/>
-<wire x1="114.3" y1="73.66" x2="121.92" y2="73.66" width="0.1524" layer="91"/>
-<wire x1="121.92" y1="73.66" x2="121.92" y2="53.34" width="0.1524" layer="91"/>
-<pinref part="FS_TF" gate="G$1" pin="2"/>
-<wire x1="121.92" y1="53.34" x2="121.92" y2="22.86" width="0.1524" layer="91"/>
-<wire x1="121.92" y1="22.86" x2="114.3" y2="22.86" width="0.1524" layer="91"/>
-<pinref part="C1_IN" gate="A" pin="6"/>
-<wire x1="142.24" y1="53.34" x2="121.92" y2="53.34" width="0.1524" layer="91"/>
-<junction x="121.92" y="53.34"/>
-</segment>
-</net>
+<wire x1="116.84" y1="71.12" x2="116.84" y2="53.34" width="0.1524" layer="91"/>
+<junction x="116.84" y="53.34"/>
+</segment>
+</net>
+<net name="N$3" class="0">
+<segment>
+<pinref part="R1_TF" gate="G$1" pin="2"/>
+<wire x1="116.84" y1="81.28" x2="116.84" y2="83.82" width="0.1524" layer="91"/>
+<pinref part="V_SUPPLY" gate="G$1" pin="1"/>
+<pinref part="R3" gate="G$1" pin="2"/>
+<wire x1="35.56" y1="91.44" x2="35.56" y2="83.82" width="0.1524" layer="91"/>
+<pinref part="R1_LF" gate="G$1" pin="2"/>
+<wire x1="35.56" y1="83.82" x2="35.56" y2="81.28" width="0.1524" layer="91"/>
+<wire x1="53.34" y1="81.28" x2="53.34" y2="83.82" width="0.1524" layer="91"/>
+<wire x1="53.34" y1="83.82" x2="35.56" y2="83.82" width="0.1524" layer="91"/>
+<junction x="35.56" y="83.82"/>
+<pinref part="R1_RF" gate="G$1" pin="2"/>
+<wire x1="68.58" y1="81.28" x2="68.58" y2="83.82" width="0.1524" layer="91"/>
+<wire x1="68.58" y1="83.82" x2="53.34" y2="83.82" width="0.1524" layer="91"/>
+<junction x="53.34" y="83.82"/>
+<pinref part="R1_MF" gate="G$1" pin="2"/>
+<wire x1="83.82" y1="81.28" x2="83.82" y2="83.82" width="0.1524" layer="91"/>
+<wire x1="83.82" y1="83.82" x2="68.58" y2="83.82" width="0.1524" layer="91"/>
+<junction x="68.58" y="83.82"/>
+<pinref part="R1_IF" gate="G$1" pin="2"/>
+<wire x1="99.06" y1="81.28" x2="99.06" y2="83.82" width="0.1524" layer="91"/>
+<junction x="83.82" y="83.82"/>
+<wire x1="99.06" y1="83.82" x2="83.82" y2="83.82" width="0.1524" layer="91"/>
+<wire x1="116.84" y1="83.82" x2="99.06" y2="83.82" width="0.1524" layer="91"/>
+<junction x="99.06" y="83.82"/>
+</segment>
+</net>

Commit message: Board created for Wheatstone bridge side
Parts:
- removed C1_IN: (no value), pinhead:PINHD-1X6
- added GND, JP1, JP2, JP3, JP4, JP5, JP6: (no value), pinhead:PINHD-1X1
Connections:
- net N$3 renamed VCC
- net GND: now also GND.1
- net N$2: now also JP1.1; no longer C1_IN.1
- net N$4: now also JP2.1; no longer C1_IN.2
- net N$6: now also JP6.1; no longer C1_IN.6
- net N$7: now also JP3.1; no longer C1_IN.3
- net N$8: now also JP4.1; no longer C1_IN.4
- net N$9: now also JP5.1; no longer C1_IN.5
Other:
- moved on the sheet: V_SUPPLY
