File: test/avneesh_test_files/Eagle_CAD/Flex_sensor_circuits/Eagle/Instrumentation_amplifier_CC3220SF.brd (EAGLE design)
At the start: 160 x 100 mm, 16 parts, among them IC1 LM324N, IC2 4051N

Commit message: Made changes to the CAD files
Parts:
- moved OUT 1.27 mm to (74.9, 45.7)
Routing:
- net N$10: track 18.3 -> 19.0 mm
Changed lines of the file:
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@@
 <attribute name="VALUE" x="49.53" y="29.845" size="1.27" layer="27"/>
 </element>
-<element name="OUT" library="pinhead" library_urn="urn:adsk.eagle:library:325" package="1X01" package3d_urn="urn:adsk.eagle:package:22485/2" value="" x="76.2" y="45.72" smashed="yes">
-<attribute name="NAME" x="74.8538" y="47.5488" size="1.27" layer="25" ratio="10"/>
-<attribute name="VALUE" x="74.93" y="42.545" size="1.27" layer="27"/>
+<element name="OUT" library="pinhead" library_urn="urn:adsk.eagle:library:325" package="1X01" package3d_urn="urn:adsk.eagle:package:22485/2" value="" x="74.93" y="45.72" smashed="yes">
+<attribute name="NAME" x="73.5838" y="47.5488" size="1.27" layer="25" ratio="10"/>
+<attribute name="VALUE" x="73.66" y="42.545" size="1.27" layer="27"/>
 </element>
 <element name="RB1" library="rcl" library_urn="urn:adsk.eagle:library:334" package="0204/7" package3d_urn="urn:adsk.eagle:package:23498/2" value="6.8 kΩ" x="58.42" y="24.13" smashed="yes" rot="R90">
@@
 <contactref element="IC1" pad="1"/>
 <contactref element="OUT" pad="1"/>
-<wire x1="76.2" y1="45.72" x2="76.2" y2="34.29" width="0.1524" layer="16"/>
-<wire x1="76.2" y1="34.29" x2="74.93" y2="33.02" width="0.1524" layer="16"/>
+<wire x1="74.93" y1="45.72" x2="74.93" y2="33.02" width="0.1524" layer="16"/>
 <wire x1="80.01" y1="45.72" x2="80.01" y2="44.45" width="0.1524" layer="16"/>
-<wire x1="80.01" y1="45.72" x2="76.2" y2="45.72" width="0.1524" layer="16"/>
+<wire x1="80.01" y1="45.72" x2="74.93" y2="45.72" width="0.1524" layer="16"/>
 </signal>
 <signal name="N$7">
